Commit message: Set up Gazebo simulation and ros2_control for mecanum robot
- Added mecanum_controllers.yaml for ros2_control config
- Created gazebo_control.xacro and robot_core.xacro
- Updated main URDF (robot.urdf.xacro)
- Added STL meshes for chassis and tyre
- Updated launch file for simulation (launch_sim.launch.py)
- Modified CMakeLists.txt and package.xml accordingly

File: description/robot_core.xacro (robot description, xacro)
@@ -54,13 +54,13 @@
 <link name="front_left_wheel">
   <visual>
-    <origin xyz="-0.0358 -0.023 -0.034" rpy="1.5709 0 1.5709"/>
-    <geometry>
-      <mesh filename="package://my_bot/meshes/tyre.STL" scale="0.001 0.001 0.001"/>
-    </geometry>
-  </visual>
-  <collision>
-    <origin xyz="-0.0358 -0.023 -0.034" rpy="1.5709 0 1.5709"/>
-    <geometry>
-      <mesh filename="package://my_bot/meshes/tyre.STL" scale="0.001 0.001 0.001"/>
+    <origin xyz="-0.0358 0.0172 -0.034" rpy="1.5709 0 1.5709"/>
+    <geometry>
+      <mesh filename="package://my_bot/meshes/tyre.STL" scale="-0.001 0.001 0.001"/>
+    </geometry>
+  </visual>
+  <collision>
+    <origin xyz="-0.0358 0.0172 -0.034" rpy="1.5709 0 1.5709"/>
+    <geometry>
+      <mesh filename="package://my_bot/meshes/tyre.STL" scale="-0.001 0.001 0.001"/>
     </geometry>
     <surface>
@@ -183,13 +183,13 @@
 <link name="rear_right_wheel">
   <visual>
-    <origin xyz="-0.0358 0.023 -0.034" rpy="0 0 -1.5709"/>
-    <geometry>
-      <mesh filename="package://my_bot/meshes/tyre.STL" scale="0.001 0.001 0.001"/>
-    </geometry>
-  </visual>
-  <collision>
-    <origin xyz="-0.0358 0.023 -0.034" rpy="0 0 -1.5709"/>
-    <geometry>
-      <mesh filename="package://my_bot/meshes/tyre.STL" scale="0.001 0.001 0.001"/>
+    <origin xyz="-0.0358 -0.0172 -0.034" rpy="0 0 -1.5709"/>
+    <geometry>
+      <mesh filename="package://my_bot/meshes/tyre.STL" scale="-0.001 0.001 0.001"/>
+    </geometry>
+  </visual>
+  <collision>
+    <origin xyz="-0.0358 -0.0172 -0.034" rpy="0 0 -1.5709"/>
+    <geometry>
+      <mesh filename="package://my_bot/meshes/tyre.STL" scale="-0.001 0.001 0.001"/>
     </geometry>
     <surface>
